Commit message: add

File: husky_description/urdf/husky.urdf.xacro (robot description, xacro)
@@ -49,5 +49,5 @@
         <origin xyz="0 0 ${height_offset}" rpy="0 0 0" />
         <geometry>
-          <!--mesh filename="package://husky_description/meshes/box3.dae" /-->
+          <mesh filename="package://husky_description/meshes/box5.dae" />
           <!--box size="${base_x_size-0.2} ${base_y_size-0.1} ${base_z_size/2 + height_offset+0.1}"/-->
         </geometry>
