Commit message: model update

File: husky_description/urdf/decorations.urdf.xacro (robot description, xacro)
@@ -22,9 +22,11 @@
 -->
 <robot name="husky_decorations" xmlns:xacro="http://ros.org/wiki/xacro">
+  <xacro:property name="height_offset" value="0.1" />
   <xacro:macro name="husky_decorate">
-    <!-- Spawn Husky chassis -->
+<!--
+    <Spawn Husky chassis >
     <link name="top_chassis_link">
       <visual>
-        <origin xyz="0 0 0" rpy="0 0 0" />
+        <origin xyz="0 0 ${height_offset}" rpy="0 0 0" />
         <geometry>
           <mesh filename="package://husky_description/meshes/top_chassis.dae" />
@@ -32,72 +34,90 @@
       </visual>
     </link>
-    <!-- Attach chassis to the robot -->
+    <Attach chassis to the robot >
     <joint name="top_chassis_joint" type="fixed">
       <parent link="base_link" />
       <child link="top_chassis_link" />
     </joint>
-    <!-- Spawn user rails -->
-    <link name="user_rail_link">
-      <visual>
-        <geometry>
-          <mesh filename="package://husky_description/meshes/user_rail.dae" />
-        </geometry>
-      </visual>
-    </link>
-    <!-- Attach user rails to base link -->
-    <joint name="user_rail" type="fixed">
-      <origin xyz="0.272 0 0.245" rpy="0 0 0" />
-      <parent link="base_link" />
-      <child link="user_rail_link" />
-    </joint>
-    <!-- Spawn front bumper link -->
-    <link name="front_bumper_link">
-      <visual>
-        <geometry>
-          <mesh filename="package://husky_description/meshes/bumper.dae" />
-        </geometry>
-      </visual>
-    </link>
-    <!-- Attach front bumper -->
-    <joint name="front_bumper" type="fixed">
-      <origin xyz="0.48 0 0.091" rpy="0 0 0" />
-      <parent link="base_link" />
-      <child link="front_bumper_link" />
-    </joint>
-    <!-- Spawn rear bumper link -->
-    <link name="rear_bumper_link">
-      <visual>
-        <geometry>
-          <mesh filename="package://husky_description/meshes/bumper.dae" />
-        </geometry>
-      </visual>
-    </link>
-    <!-- Attach rear bumper -->
-    <joint name="rear_bumper" type="fixed">
-      <origin xyz="-0.48 0 0.091" rpy="0 0 ${M_PI}" />
-      <parent link="base_link" />
-      <child link="rear_bumper_link" />
-    </joint>
+    <xacro:if value="$(optenv HUSKY_USER_RAIL_ENABLED true)">
+      <Spawn user rails >
+      <link name="user_rail_link">
+        <visual>
+          <geometry>
+            <mesh filename="package://husky_description/meshes/user_rail.dae" />
+          </geometry>
+        </visual>
+      </link>
+      <Attach user rails to base link >
+      <joint name="user_rail" type="fixed">
+        <origin xyz="0.272 0 ${height_offset+0.245}" rpy="0 0 0" />
+        <parent link="base_link" />
+        <child link="user_rail_link" />
+      </joint>
+    </xacro:if>
+-->
+    <xacro:if value="$(optenv HUSKY_FRONT_BUMPER_ENABLED true)">
+      <!-- Spawn front bumper link -->
+      <link name="front_bumper_link">
+        <visual>
+          <geometry>
+            <mesh filename="package://husky_description/meshes/bumper.dae" />
+          </geometry>
+        </visual>
+      </link>
+      <!-- Attach front bumper -->
+      <joint name="front_bumper" type="fixed">
+        <origin xyz="0.48 0 0.091" rpy="0 0 0" />
+        <parent link="base_link" />
+        <child link="front_bumper_link" />
+      </joint>
+    </xacro:if>
+    <xacro:if value="$(optenv HUSKY_REAR_BUMPER_ENABLED true)">
+      <!-- Spawn rear bumper link -->
+      <link name="rear_bumper_link">
+        <visual>
+          <geometry>
+            <mesh filename="package://husky_description/meshes/bumper.dae" />
+          </geometry>
+        </visual>
+      </link>
+      <!-- Attach rear bumper -->
+      <joint name="rear_bumper" type="fixed">
+        <origin xyz="-0.48 0 0.091" rpy="0 0 ${M_PI}" />
+        <parent link="base_link" />
+        <child link="rear_bumper_link" />
+      </joint>
+    </xacro:if>
     <xacro:if value="$(optenv HUSKY_TOP_PLATE_ENABLED true)">
       <!-- Spawn the top plate -->
       <link name="top_plate_link">
+<!--
+	<inertial>
+    		<origin rpy="-0.2 0 ${height_offset+0.25}" xyz="-0.2 0 0"/>
+    		<mass value="20.0"/>
+    		<inertia ixx="0.004878" ixy="-6.2341e-07" ixz="-7.4538e-07" iyy="0.00090164" iyz="-0.00014394" izz="0.0042946"/>
+  	</inertial>
         <visual>
-          <origin xyz="0 0 0" rpy="0 0 0" />
+          <!origin xyz="-0.2 0 0" rpy="0 0 0"/>
+	  <origin xyz="-0.2 0 ${height_offset+0.25}" rpy="0 0 0"/>
           <geometry>
-            <mesh filename="package://husky_description/meshes/top_plate.dae" />
+            <box size="0.52 0.41 0.5" rpy="0 0 0"/>
+            <!<mesh filename="package://husky_description/meshes/top_plate.dae" />
           </geometry>
         </visual>
         <collision>
-          <origin xyz="0 0 0" rpy="0 0 0"/>
+          <!origin xyz="-0.2 0 0" rpy="0 0 0"/>
+	  <origin xyz="-0.2 0 ${height_offset+0.25}" rpy="0 0 0"/>
           <geometry>
-            <mesh filename="package://husky_description/meshes/top_plate.dae" />
+            <box size="0.52 0.41 0.5" rpy="0 0 0"/>
+            <!<mesh filename="package://husky_description/meshes/top_plate.dae" />
           </geometry>
         </collision>
         <collision>
-          <!-- Extra collision tag for widgets on top plate -->
+          <! Extra collision tag for widgets on top plate >
           <geometry>
             <box size="0.32 0.41 0.09" rpy="0 0 0"/>
           </geometry>
         </collision>
+-->
       </link>
       <!-- Attach top plate -->

File: husky_description/urdf/husky.urdf.xacro (robot description, xacro)
@@ -22,4 +22,5 @@
 -->
 <robot name="husky_robot" xmlns:xacro="http://ros.org/wiki/xacro">
+  <xacro:include filename="$(find velodyne_description)/urdf/VLP-16.urdf.xacro"/>
   <!-- Included URDF/XACRO Files -->
   <xacro:include filename="$(find husky_description)/urdf/decorations.urdf.xacro" />
@@ -41,16 +42,47 @@
   <xacro:property name="wheel_length" value="0.1143" />
   <xacro:property name="wheel_radius" value="0.1651" />
+  <xacro:property name="height_offset" value="0.1" />
   <xacro:macro name="husky_robot">
     <!-- Base link is the center of the robot's bottom plate -->
     <link name="base_link">
       <visual>
-        <origin xyz="0 0 0" rpy="0 0 0" />
-        <geometry>
-          <mesh filename="package://husky_description/meshes/base_link.dae" />
-        </geometry>
+        <origin xyz="0 0 ${height_offset}" rpy="0 0 0" />
+        <geometry>
+          <!--mesh filename="package://husky_description/meshes/box3.dae" /-->
+          <!--box size="${base_x_size-0.2} ${base_y_size-0.1} ${base_z_size/2 + height_offset+0.1}"/-->
+        </geometry>
+     	<material name="Cyan">
+       	  <color rgba="0.0 0.0 1.0 1.0"/>
+     	</material>
       </visual>
       <collision>
         <origin xyz="0 0 ${base_z_size/4}" rpy="0 0 0" />
         <geometry>
+          <box size="${base_x_size*4/5} ${base_y_size} ${base_z_size/2}"/>
+        </geometry>
+      </collision>
+      <collision>
+        <origin xyz="0 0 ${base_z_size*3/4}" rpy="0 0 0" />
+        <geometry>
+          <box size="${base_x_size*4/5} ${base_y_size} ${base_z_size/2}"/>
+        </geometry>
+      </collision>
+    </link>
+<!--
+    <! Base link is the center of the robot's bottom plate >
+    <link name="base_link">
+      <visual>
+        <origin xyz="0 0 ${height_offset}" rpy="0 0 0" />
+        <geometry>
+          <!mesh filename="package://husky_description/meshes/base_link.dae" />
+          <box size="${base_x_size-0.2} ${base_y_size-0.1} ${base_z_size/2 + height_offset}"/>
+        </geometry>
+     	<material name="Cyan">
+       	  <color rgba="0.5 0.8 1.0 0.0"/>
+     	</material>
+      </visual>
+      <collision>
+        <origin xyz="0 0 ${base_z_size/4}" rpy="0 0 0" />
+        <geometry>
           <box size="${base_x_size} ${base_y_size} ${base_z_size/2}"/>
         </geometry>
@@ -63,4 +95,5 @@
       </collision>
     </link>
+-->
     <!-- Base footprint is on the ground under the robot -->
     <link name="base_footprint"/>
@@ -73,7 +106,9 @@
     <link name="inertial_link">
       <inertial>
-        <mass value="46.034"/>
-        <origin xyz="-0.00065 -0.085 0.062" />
-        <inertia ixx="0.6022" ixy="-0.02364" ixz="-0.1197" iyy="1.7386" iyz="-0.001544" izz="2.0296" />
+        <mass value="46.03"/>
+        <!--origin xyz="-0.00065 -0.085 0.062" /-->
+        <origin xyz="0 0 0" />
+        <!--inertia ixx="1.2022" ixy="-0.02364" ixz="-0.1197" iyy="1.4386" iyz="-0.001544" izz="5.3296" /-->
+        <inertia ixx="1" ixy="0" ixz="0" iyy="1" iyz="0" izz="1" />
       </inertial>
     </link>
@@ -93,4 +128,39 @@
     <gazebo reference="imu_link">
     </gazebo>
+ <!--
+  < Base Link >
+    <joint name="footprint1" type="fixed" >
+     <parent link="base_link" />
+      <child link="velo" />
+    </joint>
+    <link name="velo" >
+      <visual>
+        <geometry>
+          <box size="0.5 0.5 0.05" />
+        </geometry>
+      </visual>
+      <collision>
+        <geometry>
+          <box size="0.5 0.5 0.05" />
+        </geometry>
+      </collision>
+      <inertial>
+       <origin xyz="0 0 0"/>
+       <mass value="10"/>
+       <inertia ixx="3.0" ixy="0.0" ixz="0.0"
+               iyy="3.0" iyz="0.0"
+               izz="3.0" />
+      </inertial>
+    </link>
+       <mass value="0.00001"/>
+       <inertia ixx="0.0001" ixy="0.0" ixz="0.0"
+               iyy="0.0001" iyz="0.0"
+               izz="0.0001" />
+      </inertial>
+    </link>
+    <VLP-16 parent="velo" name="velodyne" topic="/velodyne_points" hz="10" samples="440">
+      <origin xyz="0.3 0 0.25" rpy="0 0 0" />
+    </VLP-16>
+-->
     <!-- Husky wheel macros -->
     <xacro:husky_wheel wheel_prefix="front_left">
@@ -132,5 +202,5 @@
       </xacro:sensor_arch>
       <joint name="kinect_frame_joint" type="fixed">
-        <origin xyz="$(optenv HUSKY_KINECT_XYZ 0 0 0)" rpy="$(optenv HUSKY_KINECT_RPY 0 0.18 3.14)" />
+        <origin xyz="$(optenv HUSKY_KINECT_XYZ 0 0 0)" rpy="$(optenv HUSKY_KINECT_RPY 0 0.0 3.14)" />
         <parent link="sensor_arch_mount_link"/>
         <child link="camera_link"/>
@@ -138,4 +208,5 @@
       <xacro:kinect_camera prefix="camera"/>
     </xacro:if>
+    <xacro:include filename="$(optenv HUSKY_URDF_EXTRAS empty.urdf)" />
   </xacro:macro>
 </robot>

File: husky_description/urdf/wheel.urdf.xacro (robot description, xacro)
@@ -27,5 +27,6 @@
 				<mass value="2.637" />
 				<origin xyz="0 0 0" />
-				<inertia  ixx="0.02467" ixy="0" ixz="0" iyy="0.04411" iyz="0" izz="0.02467" />
+				<!--<inertia  ixx="0.02467" ixy="0" ixz="0" iyy="0.04411" iyz="0" izz="0.02467" /-->
+				<inertia ixx="0.012411765597" ixy="0" ixz="0" iyy="0.015218160428" iyz="0" izz="0.011763977943" />
 			</inertial>
 			<visual>
@@ -43,6 +44,6 @@
 		</link>
 		<gazebo reference="${wheel_prefix}_wheel_link">
-			<mu1 value="1.0"/>
-			<mu2 value="1.0"/>
+			<mu1 value="0.7"/>
+			<mu2 value="0.7"/>
 			<kp value="10000000.0" />
 			<kd value="1.0" />

Commit message: add

File: husky_description/urdf/decorations.urdf.xacro (robot description, xacro)
@@ -22,11 +22,9 @@
 -->
 <robot name="husky_decorations" xmlns:xacro="http://ros.org/wiki/xacro">
-  <xacro:property name="height_offset" value="0.1" />
   <xacro:macro name="husky_decorate">
-<!--
-    <Spawn Husky chassis >
+    <!-- Spawn Husky chassis -->
     <link name="top_chassis_link">
       <visual>
-        <origin xyz="0 0 ${height_offset}" rpy="0 0 0" />
+        <origin xyz="0 0 0" rpy="0 0 0" />
         <geometry>
           <mesh filename="package://husky_description/meshes/top_chassis.dae" />
@@ -34,5 +32,5 @@
       </visual>
     </link>
-    <Attach chassis to the robot >
+    <!-- Attach chassis to the robot -->
     <joint name="top_chassis_joint" type="fixed">
       <parent link="base_link" />
@@ -40,5 +38,5 @@
     </joint>
     <xacro:if value="$(optenv HUSKY_USER_RAIL_ENABLED true)">
-      <Spawn user rails >
+      <!-- Spawn user rails -->
       <link name="user_rail_link">
         <visual>
@@ -48,12 +46,11 @@
         </visual>
       </link>
-      <Attach user rails to base link >
+      <!-- Attach user rails to base link -->
       <joint name="user_rail" type="fixed">
-        <origin xyz="0.272 0 ${height_offset+0.245}" rpy="0 0 0" />
+        <origin xyz="0.272 0 0.245" rpy="0 0 0" />
         <parent link="base_link" />
         <child link="user_rail_link" />
       </joint>
     </xacro:if>
--->
     <xacro:if value="$(optenv HUSKY_FRONT_BUMPER_ENABLED true)">
       <!-- Spawn front bumper link -->
@@ -91,33 +88,22 @@
       <!-- Spawn the top plate -->
       <link name="top_plate_link">
-<!--
-	<inertial>
-    		<origin rpy="-0.2 0 ${height_offset+0.25}" xyz="-0.2 0 0"/>
-    		<mass value="20.0"/>
-    		<inertia ixx="0.004878" ixy="-6.2341e-07" ixz="-7.4538e-07" iyy="0.00090164" iyz="-0.00014394" izz="0.0042946"/>
-  	</inertial>
         <visual>
-          <!origin xyz="-0.2 0 0" rpy="0 0 0"/>
-	  <origin xyz="-0.2 0 ${height_offset+0.25}" rpy="0 0 0"/>
+          <origin xyz="0 0 0" rpy="0 0 0" />
           <geometry>
-            <box size="0.52 0.41 0.5" rpy="0 0 0"/>
-            <!<mesh filename="package://husky_description/meshes/top_plate.dae" />
+            <mesh filename="package://husky_description/meshes/top_plate.dae" />
           </geometry>
         </visual>
         <collision>
-          <!origin xyz="-0.2 0 0" rpy="0 0 0"/>
-	  <origin xyz="-0.2 0 ${height_offset+0.25}" rpy="0 0 0"/>
+          <origin xyz="0 0 0" rpy="0 0 0"/>
           <geometry>
-            <box size="0.52 0.41 0.5" rpy="0 0 0"/>
-            <!<mesh filename="package://husky_description/meshes/top_plate.dae" />
+            <mesh filename="package://husky_description/meshes/top_plate.dae" />
           </geometry>
         </collision>
         <collision>
-          <! Extra collision tag for widgets on top plate >
+          <!-- Extra collision tag for widgets on top plate -->
           <geometry>
             <box size="0.32 0.41 0.09" rpy="0 0 0"/>
           </geometry>
         </collision>
--->
       </link>
       <!-- Attach top plate -->

File: husky_description/urdf/husky.urdf.xacro (robot description, xacro)
@@ -22,5 +22,4 @@
 -->
 <robot name="husky_robot" xmlns:xacro="http://ros.org/wiki/xacro">
-  <xacro:include filename="$(find velodyne_description)/urdf/VLP-16.urdf.xacro"/>
   <!-- Included URDF/XACRO Files -->
   <xacro:include filename="$(find husky_description)/urdf/decorations.urdf.xacro" />
@@ -42,43 +41,12 @@
   <xacro:property name="wheel_length" value="0.1143" />
   <xacro:property name="wheel_radius" value="0.1651" />
-  <xacro:property name="height_offset" value="0.1" />
   <xacro:macro name="husky_robot">
     <!-- Base link is the center of the robot's bottom plate -->
     <link name="base_link">
       <visual>
-        <origin xyz="0 0 ${height_offset}" rpy="0 0 0" />
+        <origin xyz="0 0 0" rpy="0 0 0" />
         <geometry>
-          <mesh filename="package://husky_description/meshes/box5.dae" />
-          <!--box size="${base_x_size-0.2} ${base_y_size-0.1} ${base_z_size/2 + height_offset+0.1}"/-->
+          <mesh filename="package://husky_description/meshes/base_link.dae" />
         </geometry>
-     	<material name="Cyan">
-       	  <color rgba="0.0 0.0 1.0 1.0"/>
-     	</material>
-      </visual>
-      <collision>
-        <origin xyz="0 0 ${base_z_size/4}" rpy="0 0 0" />
-        <geometry>
-          <box size="${base_x_size*4/5} ${base_y_size} ${base_z_size/2}"/>
-        </geometry>
-      </collision>
-      <collision>
-        <origin xyz="0 0 ${base_z_size*3/4}" rpy="0 0 0" />
-        <geometry>
-          <box size="${base_x_size*4/5} ${base_y_size} ${base_z_size/2}"/>
-        </geometry>
-      </collision>
-    </link>
-<!--
-    <! Base link is the center of the robot's bottom plate >
-    <link name="base_link">
-      <visual>
-        <origin xyz="0 0 ${height_offset}" rpy="0 0 0" />
-        <geometry>
-          <!mesh filename="package://husky_description/meshes/base_link.dae" />
-          <box size="${base_x_size-0.2} ${base_y_size-0.1} ${base_z_size/2 + height_offset}"/>
-        </geometry>
-     	<material name="Cyan">
-       	  <color rgba="0.5 0.8 1.0 0.0"/>
-     	</material>
       </visual>
       <collision>
@@ -95,5 +63,4 @@
       </collision>
     </link>
--->
     <!-- Base footprint is on the ground under the robot -->
     <link name="base_footprint"/>
@@ -106,9 +73,7 @@
     <link name="inertial_link">
       <inertial>
-        <mass value="46.03"/>
-        <!--origin xyz="-0.00065 -0.085 0.062" /-->
-        <origin xyz="0 0 0" />
-        <!--inertia ixx="1.2022" ixy="-0.02364" ixz="-0.1197" iyy="1.4386" iyz="-0.001544" izz="5.3296" /-->
-        <inertia ixx="1" ixy="0" ixz="0" iyy="1" iyz="0" izz="1" />
+        <mass value="46.034"/>
+        <origin xyz="-0.00065 -0.085 0.062" />
+        <inertia ixx="0.6022" ixy="-0.02364" ixz="-0.1197" iyy="1.7386" iyz="-0.001544" izz="2.0296" />
       </inertial>
     </link>
@@ -128,39 +93,4 @@
     <gazebo reference="imu_link">
     </gazebo>
- <!--
-  < Base Link >
-    <joint name="footprint1" type="fixed" >
-     <parent link="base_link" />
-      <child link="velo" />
-    </joint>
-    <link name="velo" >
-      <visual>
-        <geometry>
-          <box size="0.5 0.5 0.05" />
-        </geometry>
-      </visual>
-      <collision>
-        <geometry>
-          <box size="0.5 0.5 0.05" />
-        </geometry>
-      </collision>
-      <inertial>
-       <origin xyz="0 0 0"/>
-       <mass value="10"/>
-       <inertia ixx="3.0" ixy="0.0" ixz="0.0"
-               iyy="3.0" iyz="0.0"
-               izz="3.0" />
-      </inertial>
-    </link>
-       <mass value="0.00001"/>
-       <inertia ixx="0.0001" ixy="0.0" ixz="0.0"
-               iyy="0.0001" iyz="0.0"
-               izz="0.0001" />
-      </inertial>
-    </link>
-    <VLP-16 parent="velo" name="velodyne" topic="/velodyne_points" hz="10" samples="440">
-      <origin xyz="0.3 0 0.25" rpy="0 0 0" />
-    </VLP-16>
--->
     <!-- Husky wheel macros -->
     <xacro:husky_wheel wheel_prefix="front_left">
@@ -202,5 +132,5 @@
       </xacro:sensor_arch>
       <joint name="kinect_frame_joint" type="fixed">
-        <origin xyz="$(optenv HUSKY_KINECT_XYZ 0 0 0)" rpy="$(optenv HUSKY_KINECT_RPY 0 0.0 3.14)" />
+        <origin xyz="$(optenv HUSKY_KINECT_XYZ 0 0 0)" rpy="$(optenv HUSKY_KINECT_RPY 0 0.18 3.14)" />
         <parent link="sensor_arch_mount_link"/>
         <child link="camera_link"/>

File: husky_description/urdf/wheel.urdf.xacro (robot description, xacro)
@@ -27,6 +27,5 @@
 				<mass value="2.637" />
 				<origin xyz="0 0 0" />
-				<!--<inertia  ixx="0.02467" ixy="0" ixz="0" iyy="0.04411" iyz="0" izz="0.02467" /-->
-				<inertia ixx="0.012411765597" ixy="0" ixz="0" iyy="0.015218160428" iyz="0" izz="0.011763977943" />
+				<inertia  ixx="0.02467" ixy="0" ixz="0" iyy="0.04411" iyz="0" izz="0.02467" />
 			</inertial>
 			<visual>
@@ -44,6 +43,6 @@
 		</link>
 		<gazebo reference="${wheel_prefix}_wheel_link">
-			<mu1 value="0.7"/>
-			<mu2 value="0.7"/>
+			<mu1 value="1.0"/>
+			<mu2 value="1.0"/>
 			<kp value="10000000.0" />
 			<kd value="1.0" />
